File: FilamentDriver.kicad_sch (KiCad schematic)
At the start: 10 parts, among them U3 SN6507DGQ

Commit message: Rev 0.1
Connections:
- net GND: now also D2.1 (A); no longer D2.2 (A)
Changed lines of the file:
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@@
 			)
 		)
-		(pin "2"
+		(pin "1"
 		)
 		(pin "3"

Commit message: bitbanging
Connections:
- net +3.3V: now also TR1.2; no longer TR1.5
- net F1: now also TR1.4; no longer TR1.1
- net at D2.3 (K), R7.2: now also TR1.5; no longer TR1.2
- net at U3.1 (SW1): now also TR1.1; no longer TR1.4
- net at U3.10 (SW2): now also TR1.3; no longer TR1.6
- net at R8.1: now also TR1.6; no longer TR1.3
Other:
- moved on the sheet: TR1
