File: controller.kicad_sch (KiCad schematic)
At the start: 19 parts, among them J2 Micro_SD_Card_Det2, SW1 SKRKAEE020, SW2 SKRKAEE020, SW3 SKRKAEE020, U7 MN12832L, U8 STM32U073CB

Commit message: spi_pins
VFD over SPI
3.3V and 5V over P-Channel Mosfet
Parts:
- added Q5, Q6: IRLML6401, Package_TO_SOT_SMD:SOT-23, symbol Transistor_FET:IRLML6401
- added R20, R21: 10k, Resistor_SMD:R_0603_1608Metric, symbol Device:R
- added R22, R23: 100R, Resistor_SMD:R_0603_1608Metric, symbol Device:R
Connections:
- net +3.3V: now also Q6.2 (S), R21.1; no longer C21.1, J2.4 (VDD), U7.9 (VDD1)
- net CLK: now also U8.11 (PA1); no longer U8.30 (PA9)
- net SIN1: now also U8.28 (PB15); no longer U8.31 (PA10)
- net SIN2: now also U7.14 (SOUT1); no longer U8.38 (PA15)
- net SOUT2: no longer U8.28 (PB15)
- net VPMID_5V: now also Q5.2 (S), R20.1
- net SOUT1 renamed ~{3.3V_EN}
- net ~{3.3V_EN}: now also R21.2, R23.1; no longer U7.14 (SOUT1)
- new net: Q5.1 (G), R22.2
- new net: Q6.1 (G), R23.2
- new net 3.3V_SWITCHED: C21.1, J2.4 (VDD), Q6.3 (D), U7.9 (VDD1)
- new net 5V_SWITCHED: Q5.3 (D)
- new net ~{5V_EN}: R20.2, R22.1, U8.30 (PA9)
- no-connect marks 18 -> 17
